Commit message: refactor: migrate SEED-Noid to ROS2 Jazzy

File: model/parts/typeg_body/typeg_body.xacro (robot description, xacro)
@@ -41,4 +41,8 @@
          joint_effort_limit="10" />
       <link name="hip_center">
+         <inertial>
+            <mass value="0.1" />
+            <inertia ixx="0.001" ixy="0" ixz="0" iyy="0.001" iyz="0" izz="0.001" />
+         </inertial>
       </link>
       <xacro:armjoint

File: model/parts/typeg_larm/typeg_larm.xacro (robot description, xacro)
@@ -75,4 +75,8 @@
          joint_effort_limit="10" />
       <link name="l_elbow_virtual_link">
+         <inertial>
+            <mass value="0.05" />
+            <inertia ixx="0.0005" ixy="0" ixz="0" iyy="0.0005" iyz="0" izz="0.0005" />
+         </inertial>
       </link>
       <xacro:armjoint
@@ -89,4 +93,8 @@
          mimic="true" />
       <link name="l_elbow_virtual_link_dummy">
+         <inertial>
+            <mass value="0.05" />
+            <inertia ixx="0.0005" ixy="0" ixz="0" iyy="0.0005" iyz="0" izz="0.0005" />
+         </inertial>
       </link>
       <xacro:armjoint

File: model/parts/typeg_rarm/typeg_rarm.xacro (robot description, xacro)
@@ -75,4 +75,8 @@
          joint_effort_limit="10" />
       <link name="r_elbow_virtual_link">
+         <inertial>
+            <mass value="0.05" />
+            <inertia ixx="0.0005" ixy="0" ixz="0" iyy="0.0005" iyz="0" izz="0.0005" />
+         </inertial>
       </link>
       <xacro:armjoint
@@ -89,4 +93,8 @@
          mimic="true" />
       <link name="r_elbow_virtual_link_dummy">
+         <inertial>
+            <mass value="0.05" />
+            <inertia ixx="0.0005" ixy="0" ixz="0" iyy="0.0005" iyz="0" izz="0.0005" />
+         </inertial>
       </link>
       <xacro:armjoint

File: model/parts/xacro_common.xacro (robot description, xacro)
@@ -4,6 +4,12 @@
     <xacro:arg name="mesh_visual" default="mesh" />
     <xacro:arg name="mesh_collision" default="mesh" />
-    <xacro:macro name="armlink" params="link_name model_type mesh_name base_origin_xyz base_origin_rpy">
+    <!-- mass/inertiaはGazeboシミュレーション用(実機制御では未使用)。
+         重くしすぎると関節のeffort limitが飽和して腕が垂れる -->
+    <xacro:macro name="armlink" params="link_name model_type mesh_name base_origin_xyz base_origin_rpy mass:=0.2 ixx:=0.003 iyy:=0.003 izz:=0.003">
         <link name="${link_name}">
+            <inertial>
+                <mass value="${mass}" />
+                <inertia ixx="${ixx}" ixy="0" ixz="0" iyy="${iyy}" iyz="0" izz="${izz}" />
+            </inertial>
             <visual>
                 <origin xyz="${base_origin_xyz}" rpy="${base_origin_rpy}" />
